Commit message: wip ejemplo

File: code/ros2/install/pibotj_description/share/pibotj_description/urdf/caster_diffbot.xacro (robot description, xacro)
@@ -1,5 +1,5 @@
 <?xml version="1.0"?>
 <robot name="caster_diffbot" xmlns:xacro="http://ros.org/wiki/xacro">
-  <xacro:property name="package_name" value="pibotj_description"/>
+  <xacro:property name="package_name" value="basic_diffbot"/>
   <xacro:property name="PI" value="3.14159265"/>
   <xacro:property name="wheelSeparation" value="0.13"/>
@@ -16,9 +16,7 @@
   <link name="base_link"> <!-- Important: Every visual, collision and inertial tag has its own origin -->
     <visual>
-      <!--origin xyz="-0.033 0.0 0.04" rpy="0 0 ${PI}"/-->
-      <origin xyz="-0.17 -0.055 0.04" rpy="${-PI/2} 0 0"/>
+      <origin xyz="-0.033 0.0 0.04" rpy="0 0 ${PI}"/>
       <geometry>
-        <!--mesh filename="package://${package_name}/meshes/base_plate.stl" scale="1 1 1"/-->
-        <mesh filename="package://${package_name}/meshes/base.stl" scale="0.001 0.001 0.001"/>
+        <mesh filename="package://${package_name}/meshes/base_plate.stl" scale="1 1 1"/>
       </geometry>
       <material name="Blue"> <!-- Color in Rviz2 (inside visual tag) -->

File: code/ros2/install/pibotj_description/share/pibotj_description/urdf/the_simplest_diffbot.xacro (robot description, xacro)
@@ -1,5 +1,5 @@
 <?xml version="1.0"?>
 <robot name="the_simplest_diffbot" xmlns:xacro="http://ros.org/wiki/xacro">
-  <xacro:include filename="$(find pibotj_description)/urdf/the_simplest_diffbot_gz.xacro"/>
+  <xacro:include filename="$(find basic_diffbot)/urdf/the_simplest_diffbot_gz.xacro"/>
   <link name="base_footprint"/>
   <joint name="base_joint" type="fixed">
