Commit message: added camera and wip modified robot parts

File: code/ros2/install/pibotj/share/pibotj/urdf/caster_diffbot.xacro (robot description, xacro)
@@ -102,9 +102,10 @@
     <origin xyz="-0.104 0 0.015" rpy="0 0 ${PI}" />
     <parent link="base_link" />
-    <child link="caster_base_link" />
+    <!--child link="caster_base_link" /-->
+    <child link="caster_wheel_link" />
     <!--axis xyz="0 0 1" /-->
     <!--dynamics damping="0.001" fricction="0.001"/-->
   </joint>
-  <link name="caster_base_link">
+  <!--link name="caster_base_link">
     <visual>
       <origin xyz="0 0 0.015" rpy="${-PI} 0 0" />
@@ -118,11 +119,11 @@
       <inertia ixx="0.00004" ixy="0" ixz="0" iyy="0.00004" iyz="0" izz="0.00001" />
     </inertial>
-  </link>
-  <joint name="caster_wheel_joint" type="fixed">
+  </link-->
+  <!--joint name="caster_wheel_joint" type="fixed">
     <origin xyz="0.015014 -0.00012272 -0.01" rpy="0 ${-PI/2} ${PI/2}" />
     <parent link="caster_base_link" />
-    <child link="caster_wheel_link" />
+    <child link="caster_wheel_link" /-->
     <!--axis xyz="0 0 1" /-->
-  </joint>
+  <!--/joint-->
   <link name="caster_wheel_link">
     <visual>
@@ -146,12 +147,12 @@
   <!-- ******************** SENSORS DEFINITION ******************** -->
   <!-- IMU -->
-  <joint name="imu_joint" type="fixed">
+  <!--joint name="imu_joint" type="fixed">
     <parent link="base_link"/>
     <child link="imu_link"/>
     <origin xyz="0 0 0" rpy="0 0 0"/>
   </joint>
-  <link name="imu_link" />
+  <link name="imu_link" /-->
   <!-- LIDAR -->
-  <joint name="lidar_joint" type="fixed">
+  <!--joint name="lidar_joint" type="fixed">
     <parent link="base_link"/>
     <child link="lidar_link"/>
@@ -165,12 +166,12 @@
       </geometry>
     </visual>
-  </link>
+  </link-->
   <!-- CAMERA -->
   <joint name="camera_joint" type="fixed">
-    <origin xyz="0.04 0 0.05" rpy="0 0 0"/>
+    <origin xyz="0.04 0.025 0.05" rpy="0 0 0"/>
     <parent link="base_link"/>
     <child link="camera_frame"/>
   </joint>
-  <link name="camera_frame">
+  <!--link name="camera_frame">
     <visual>
       <origin xyz="0 0 0" rpy="0 0 0"/>
@@ -179,11 +180,24 @@
       </geometry>
     </visual>
-  </link>
-  <joint name="logo_joint" type="fixed">
+  </link-->
+  <link name="camera_frame"> <!-- Important: Every visual, collision and inertial tag has its own origin -->
+    <visual>
+      <!--origin xyz="-0.033 0.0 0.04" rpy="0 0 ${PI}"/-->
+      <origin xyz="0.0 0.0 0.0 " rpy="0 0 ${-PI/2}"/>
+      <geometry>
+        <!--mesh filename="package://${package_name}/meshes/base_plate.stl" scale="1 1 1"/-->
+        <mesh filename="package://${package_name}/meshes/camara.stl" scale="0.001 0.001 0.001"/>
+      </geometry>
+      <material name="Blue"> <!-- Color in Rviz2 (inside visual tag) -->
+        <color rgba="${0/255} ${0/255} ${255/255} 1.0"/>
+      </material>
+    </visual>
+  </link>
+  <!--joint name="logo_joint" type="fixed">
     <parent link="base_footprint"/>
     <child link="logo_link"/>
     <origin xyz="-0.09 0.0 0.05" rpy="0 0 0"/>
-  </joint>
-  <link name="logo_link">
+  </joint-->
+  <!--link name="logo_link">
     <visual>
       <origin xyz="0 0 0" rpy="0 0 ${PI}"/>
@@ -198,4 +212,4 @@
       </geometry>
     </collision>
-  </link>
+  </link-->
 </robot>

File: code/ros2/install/pibotj/share/pibotj/urdf/caster_diffbot_gz.xacro (robot description, xacro)
@@ -30,5 +30,5 @@
     <material>Gazebo/DarkGrey</material>
   </gazebo>
-  <gazebo reference="caster_base_link">
+  <!--gazebo reference="caster_base_link">
     <mu1>0.1</mu1>
     <mu2>0.1</mu2>
@@ -38,5 +38,5 @@
     <maxVel>1.0</maxVel>
     <material>Gazebo/$(arg base_color)</material>
-  </gazebo>
+  </gazebo-->
   <gazebo reference="caster_wheel_link">
     <mu1>0.1</mu1>
@@ -90,5 +90,5 @@
   <!-- ******************** SENSORS PLUGINS ******************** -->
   <!-- IMU -->
-  <gazebo reference="imu_link">
+  <!--gazebo reference="imu_link">
     <sensor name="imu" type="imu">
       <visualize>true</visualize>
@@ -96,7 +96,7 @@
       <update_rate>30</update_rate>
       <plugin name="imu_plugin" filename="libgazebo_ros_imu_sensor.so">
-        <ros>
+        <ros-->
           <!--namespace>/</namespace-->
-          <remapping>~/out:=imu</remapping>
+          <!--remapping>~/out:=imu</remapping>
         </ros>
         <initial_orientation_as_reference>false</initial_orientation_as_reference>
@@ -157,7 +157,7 @@
       </imu>
     </sensor>
-  </gazebo>
+  </gazebo-->
   <!-- LIDAR -->
-  <gazebo reference="lidar_link">
+  <!--gazebo reference="lidar_link">
     <material>Gazebo/Black</material>
     <sensor type="ray" name="lidar">
@@ -187,17 +187,17 @@
       </ray>
       <plugin name="laser_plugin" filename="libgazebo_ros_ray_sensor.so">
-        <ros>
+        <ros-->
             <!--namespace>/</namespace-->
-            <remapping>~/out:=scan</remapping>
-        </ros>
+            <!--remapping>~/out:=scan</remapping>
+        </ros-->
         <!--topic_name>scan</topic_name-->
-        <output_type>sensor_msgs/LaserScan</output_type>
+        <!--output_type>sensor_msgs/LaserScan</output_type>
         <frame_name>lidar_link</frame_name>
       </plugin>
     </sensor>
-  </gazebo>
+  </gazebo-->
   <!-- MONOCULAR CAMERA -->
   <gazebo reference="camera_frame">
-    <material>Gazebo/Orange</material>
+    <material>Gazebo/Blue</material>
     <sensor type="camera" name="camera">
       <always_on>true</always_on>

File: code/ros2/src/pibotj/urdf/caster_diffbot.xacro (robot description, xacro)
@@ -102,9 +102,10 @@
     <origin xyz="-0.104 0 0.015" rpy="0 0 ${PI}" />
     <parent link="base_link" />
-    <child link="caster_base_link" />
+    <!--child link="caster_base_link" /-->
+    <child link="caster_wheel_link" />
     <!--axis xyz="0 0 1" /-->
     <!--dynamics damping="0.001" fricction="0.001"/-->
   </joint>
-  <link name="caster_base_link">
+  <!--link name="caster_base_link">
     <visual>
       <origin xyz="0 0 0.015" rpy="${-PI} 0 0" />
@@ -118,11 +119,11 @@
       <inertia ixx="0.00004" ixy="0" ixz="0" iyy="0.00004" iyz="0" izz="0.00001" />
     </inertial>
-  </link>
-  <joint name="caster_wheel_joint" type="fixed">
+  </link-->
+  <!--joint name="caster_wheel_joint" type="fixed">
     <origin xyz="0.015014 -0.00012272 -0.01" rpy="0 ${-PI/2} ${PI/2}" />
     <parent link="caster_base_link" />
-    <child link="caster_wheel_link" />
+    <child link="caster_wheel_link" /-->
     <!--axis xyz="0 0 1" /-->
-  </joint>
+  <!--/joint-->
   <link name="caster_wheel_link">
     <visual>
@@ -146,12 +147,12 @@
   <!-- ******************** SENSORS DEFINITION ******************** -->
   <!-- IMU -->
-  <joint name="imu_joint" type="fixed">
+  <!--joint name="imu_joint" type="fixed">
     <parent link="base_link"/>
     <child link="imu_link"/>
     <origin xyz="0 0 0" rpy="0 0 0"/>
   </joint>
-  <link name="imu_link" />
+  <link name="imu_link" /-->
   <!-- LIDAR -->
-  <joint name="lidar_joint" type="fixed">
+  <!--joint name="lidar_joint" type="fixed">
     <parent link="base_link"/>
     <child link="lidar_link"/>
@@ -165,12 +166,12 @@
       </geometry>
     </visual>
-  </link>
+  </link-->
   <!-- CAMERA -->
   <joint name="camera_joint" type="fixed">
-    <origin xyz="0.04 0 0.05" rpy="0 0 0"/>
+    <origin xyz="0.04 0.025 0.05" rpy="0 0 0"/>
     <parent link="base_link"/>
     <child link="camera_frame"/>
   </joint>
-  <link name="camera_frame">
+  <!--link name="camera_frame">
     <visual>
       <origin xyz="0 0 0" rpy="0 0 0"/>
@@ -179,11 +180,24 @@
       </geometry>
     </visual>
-  </link>
-  <joint name="logo_joint" type="fixed">
+  </link-->
+  <link name="camera_frame"> <!-- Important: Every visual, collision and inertial tag has its own origin -->
+    <visual>
+      <!--origin xyz="-0.033 0.0 0.04" rpy="0 0 ${PI}"/-->
+      <origin xyz="0.0 0.0 0.0 " rpy="0 0 ${-PI/2}"/>
+      <geometry>
+        <!--mesh filename="package://${package_name}/meshes/base_plate.stl" scale="1 1 1"/-->
+        <mesh filename="package://${package_name}/meshes/camara.stl" scale="0.001 0.001 0.001"/>
+      </geometry>
+      <material name="Blue"> <!-- Color in Rviz2 (inside visual tag) -->
+        <color rgba="${0/255} ${0/255} ${255/255} 1.0"/>
+      </material>
+    </visual>
+  </link>
+  <!--joint name="logo_joint" type="fixed">
     <parent link="base_footprint"/>
     <child link="logo_link"/>
     <origin xyz="-0.09 0.0 0.05" rpy="0 0 0"/>
-  </joint>
-  <link name="logo_link">
+  </joint-->
+  <!--link name="logo_link">
     <visual>
       <origin xyz="0 0 0" rpy="0 0 ${PI}"/>
@@ -198,4 +212,4 @@
       </geometry>
     </collision>
-  </link>
+  </link-->
 </robot>

Commit message: wip camara revolute, works fixed

File: code/ros2/install/pibotj/share/pibotj/urdf/caster_diffbot.xacro (robot description, xacro)
@@ -3,4 +3,8 @@
   <xacro:property name="package_name" value="pibotj"/>
   <xacro:property name="PI" value="3.14159265"/>
+  <!--xacro:property name="wheelSeparation" value="0.13"/>
+  <xacro:property name="wheelDiameter" value="0.07"/>
+  <xacro:property name="wheelThickness" value="0.024"/>
+  <xacro:property name="base_elevation" value="0.01"/-->
   <xacro:property name="wheelSeparation" value="0.13"/>
   <xacro:property name="wheelDiameter" value="0.07"/>
@@ -100,5 +104,6 @@
   <!-- Caster wheel definition (joints and links) -->
   <joint name="caster_base_joint" type="fixed">
-    <origin xyz="-0.104 0 0.015" rpy="0 0 ${PI}" />
+    <!--origin xyz="-0.104 0 0.015" rpy="0 0 ${PI}" /-->
+    <origin xyz="-0.135 -0.01 0.006" rpy="0 ${PI} ${PI}" />
     <parent link="base_link" />
     <!--child link="caster_base_link" /-->
@@ -130,5 +135,5 @@
       <origin xyz="0 0 0" rpy="0 0 0" />
       <geometry>
-        <mesh filename="package://${package_name}/meshes/caster_wheel.stl" />
+        <mesh filename="package://${package_name}/meshes/bolaloca.stl" scale="0.001 0.001 0.001"/>
       </geometry>
     </visual>
@@ -136,5 +141,6 @@
       <origin xyz="0 0 0" rpy="0 0 0" />
       <geometry>
-        <cylinder length="0.01" radius="0.015" />
+        <!--cylinder length="0.01" radius="0.015" /-->
+        <box size="0.01 0.1 0.03"/>
       </geometry>
     </collision>
@@ -173,4 +179,12 @@
     <child link="camera_frame"/>
   </joint>
+  <!--joint name="camera_joint" type="revolute">
+    <origin xyz="0.04 0.025 0.05" rpy="0 0 0"/>
+    <parent link="base_link"/>
+    <child link="camera_frame"/>
+    <axis xyz="0 1 0"/>
+    <limit effort="1.0" lower="0" upper="3.14159" velocity="0.5"/>
+  <dynamics damping="0.5" friction="0.5"/>
+  </joint-->
   <!--link name="camera_frame">
     <visual>
@@ -193,4 +207,17 @@
       </material>
     </visual>
+    <!-- NECESARIO AÑADIRLO PARA QUE GAZEBO NO NOS IGNORE-->
+    <!-- Collision tag added to stabilize the robot -->
+    <!--collision>
+      <origin xyz="0.0 0.0 0.0 " rpy="0 0 ${-PI/2}"/>
+      <geometry-->
+        <!--mesh filename="package://${package_name}/meshes/base_plate.stl" scale="1 1 1"/-->
+        <!--mesh filename="package://${package_name}/meshes/camara.stl" scale="0.001 0.001 0.001"/>
+      </geometry>
+    </collision>
+    <inertial>
+      <origin xyz="0.0 0.0 0.0" rpy="0 0 ${-PI/2}"/>
+        <inertia ixx="0.0011" ixy="0" ixz="0" iyy="0.0084" iyz="0" izz="0.0011" />
+      </inertial-->
   </link>
   <!--joint name="logo_joint" type="fixed">

File: code/ros2/install/pibotj/share/pibotj/urdf/caster_diffbot_gz.xacro (robot description, xacro)
@@ -46,5 +46,5 @@
     <minDepth>0.001</minDepth>
     <maxVel>1.0</maxVel>
-    <material>Gazebo/Black</material>
+    <material>Gazebo/White</material>
   </gazebo>
   <!-- Plugins for a differential drive mobile robot in Gazebo with ROS 2 -->
@@ -198,5 +198,16 @@
   </gazebo-->
   <!-- MONOCULAR CAMERA -->
-  <gazebo reference="camera_frame">
+<!--gazebo reference="camera_joint">
+  <plugin name="camera_joint_control" filename="libgazebo_ros_joint_control.so">
+    <ros>
+      <namespace>/</namespace>
+      <remapping>~/command:=camera_joint/command</remapping>
+    </ros>
+    <joint_name>camera_joint</joint_name>
+    <update_rate>30</update_rate-->
+    <!-- Configura otros parámetros según sea necesario -->
+  <!--/plugin>
+</gazebo-->
+  <!--gazebo reference="camera_frame">
     <material>Gazebo/Blue</material>
     <sensor type="camera" name="camera">
@@ -225,7 +236,7 @@
       </camera>
         <plugin name="camera_plugin" filename="libgazebo_ros_camera.so">
-            <ros>
+            <ros-->
                 <!--namespace>/</namespace-->
-                <remapping>~/image_raw:=image_raw</remapping>
+                <!--remapping>~/image_raw:=image_raw</remapping>
                 <remapping>~/camera_info:=camera_info</remapping>
             </ros>
@@ -235,4 +246,4 @@
         </plugin>
     </sensor>
-  </gazebo>
+  </gazebo-->
 </robot>

Commit message: working camera structure urdf r+g

File: code/ros2/install/pibotj/share/pibotj/urdf/caster_diffbot.xacro (robot description, xacro)
@@ -174,25 +174,18 @@
   </link-->
   <!-- CAMERA -->
-  <joint name="camera_joint" type="fixed">
+  <!-- ESTE FUNCIONA -->
+  <!--joint name="camera_joint" type="fixed">
     <origin xyz="0.04 0.025 0.05" rpy="0 0 0"/>
     <parent link="base_link"/>
     <child link="camera_frame"/>
-  </joint>
-  <!--joint name="camera_joint" type="revolute">
+  </joint-->
+  <joint name="camera_joint" type="revolute">
+    <parent link="base_link"/>
+    <child link="camera_frame"/>
     <origin xyz="0.04 0.025 0.05" rpy="0 0 0"/>
-    <parent link="base_link"/>
-    <child link="camera_frame"/>
     <axis xyz="0 1 0"/>
-    <limit effort="1.0" lower="0" upper="3.14159" velocity="0.5"/>
-  <dynamics damping="0.5" friction="0.5"/>
-  </joint-->
-  <!--link name="camera_frame">
-    <visual>
-      <origin xyz="0 0 0" rpy="0 0 0"/>
-      <geometry>
-        <box size="0.01 0.03 0.02"/>
-      </geometry>
-    </visual>
-  </link-->
+    <limit effort="0.0" lower="0.0" upper="0.0" velocity="0.0"/>
+    <dynamics damping="0.05" friction="0.05"/>
+  </joint>
   <link name="camera_frame"> <!-- Important: Every visual, collision and inertial tag has its own origin -->
     <visual>
@@ -209,15 +202,15 @@
     <!-- NECESARIO AÑADIRLO PARA QUE GAZEBO NO NOS IGNORE-->
     <!-- Collision tag added to stabilize the robot -->
-    <!--collision>
+    <collision>
       <origin xyz="0.0 0.0 0.0 " rpy="0 0 ${-PI/2}"/>
-      <geometry-->
-        <!--mesh filename="package://${package_name}/meshes/base_plate.stl" scale="1 1 1"/-->
-        <!--mesh filename="package://${package_name}/meshes/camara.stl" scale="0.001 0.001 0.001"/>
+      <geometry>
+        <mesh filename="package://${package_name}/meshes/camara.stl" scale="0.001 0.001 0.001"/>
       </geometry>
     </collision>
     <inertial>
       <origin xyz="0.0 0.0 0.0" rpy="0 0 ${-PI/2}"/>
-        <inertia ixx="0.0011" ixy="0" ixz="0" iyy="0.0084" iyz="0" izz="0.0011" />
-      </inertial-->
+      <mass value="0.03"/> <!--30g-->
+      <inertia ixx="0.01" ixy="0.0" ixz="0.0" iyy="0.005" iyz="0.0" izz="0.005"/>
+      </inertial>
   </link>
   <!--joint name="logo_joint" type="fixed">

File: code/ros2/install/pibotj/share/pibotj/urdf/caster_diffbot_gz.xacro (robot description, xacro)
@@ -86,4 +86,6 @@
       <joint_name>wheel_left_joint</joint_name>
       <joint_name>wheel_right_joint</joint_name>
+      <!-- camera HA SIDO NECESARIO INCLUIRLO AQUÍ SINO NO LO DETECTA RVIZ CORRECTAMENTE-->
+      <joint_name>camera_joint</joint_name>
     </plugin>
   </gazebo>
@@ -205,9 +207,8 @@
     </ros>
     <joint_name>camera_joint</joint_name>
-    <update_rate>30</update_rate-->
-    <!-- Configura otros parámetros según sea necesario -->
-  <!--/plugin>
+    <update_rate>30</update_rate>
+  </plugin>
 </gazebo-->
-  <!--gazebo reference="camera_frame">
+  <gazebo reference="camera_frame">
     <material>Gazebo/Blue</material>
     <sensor type="camera" name="camera">
@@ -236,7 +237,7 @@
       </camera>
         <plugin name="camera_plugin" filename="libgazebo_ros_camera.so">
-            <ros-->
-                <!--namespace>/</namespace-->
-                <!--remapping>~/image_raw:=image_raw</remapping>
+            <ros>
+                <namespace>/</namespace>
+                <remapping>~/image_raw:=image_raw</remapping>
                 <remapping>~/camera_info:=camera_info</remapping>
             </ros>
@@ -246,4 +247,4 @@
         </plugin>
     </sensor>
-  </gazebo-->
+  </gazebo>
 </robot>
