Commit message: working camera rotation

File: code/ros2/install/pibotj/share/pibotj/urdf/caster_diffbot.xacro (robot description, xacro)
@@ -1,176 +1 @@
-<?xml version="1.0"?>
-<robot name="caster_diffbot" xmlns:xacro="http://ros.org/wiki/xacro">
-  <xacro:property name="package_name" value="pibotj"/>
-  <xacro:property name="PI" value="3.14159265"/>
-  <!--xacro:property name="wheelSeparation" value="0.13"/>
-  <xacro:property name="wheelDiameter" value="0.07"/>
-  <xacro:property name="wheelThickness" value="0.024"/>
-  <xacro:property name="base_elevation" value="0.01"/-->
-  <xacro:property name="wheelSeparation" value="0.13"/>
-  <xacro:property name="wheelDiameter" value="0.07"/>
-  <xacro:property name="wheelThickness" value="0.024"/>
-  <xacro:property name="base_elevation" value="0.01"/>
-  <xacro:include filename="$(find ${package_name})/urdf/caster_diffbot_gz.xacro"/>
-  <link name="base_footprint"/>
-  <joint name="base_joint" type="fixed">
-    <parent link="base_footprint"/>
-    <child link="base_link"/>
-    <origin xyz="0 0 ${base_elevation}" rpy="0 0 0"/>
-  </joint>
-  <link name="base_link"> <!-- Important: Every visual, collision and inertial tag has its own origin -->
-    <visual>
-      <!--origin xyz="-0.033 0.0 0.04" rpy="0 0 ${PI}"/-->
-      <origin xyz="-0.17 -0.055 0.04" rpy="${-PI/2} 0 0"/>
-      <geometry>
-        <!--mesh filename="package://${package_name}/meshes/base_plate.stl" scale="1 1 1"/-->
-        <mesh filename="package://${package_name}/meshes/base.stl" scale="0.001 0.001 0.001"/>
-      </geometry>
-      <material name="Blue"> <!-- Color in Rviz2 (inside visual tag) -->
-        <color rgba="${0/255} ${0/255} ${255/255} 1.0"/>
-      </material>
-    </visual>
-    <collision>
-      <origin xyz="-0.17 0 0.04" rpy="0 0 0"/>
-      <geometry>
-        <box size="0.2 0.1 0.01"/>
-      </geometry>
-    </collision>
-    <!-- Collision tag added to stabilize the robot -->
-    <collision>
-      <origin xyz="0.06 0 0.002" rpy="0 0 0" />
-      <geometry>
-        <sphere radius="0.01" />
-      </geometry>
-    </collision>
-    <inertial>
-      <origin xyz="0 0 ${wheelDiameter-base_elevation}" rpy="0 0 0"/>
-      <mass value="10"/>
-      <inertia ixx="0.333333" ixy="0.0" ixz="0.0"  iyy="0.333333" iyz="0.0"  izz="0.6" />
-    </inertial>
-  </link>
-  <!-- Wheels definition (joints and links) -->
-  <joint name="wheel_left_joint" type="continuous">
-    <parent link="base_link"/>
-    <child link="wheel_left_link"/>
-    <origin xyz="0 ${wheelSeparation/2} ${wheelDiameter/2-base_elevation}" rpy="${-PI/2} 0 0"/>
-    <axis xyz="0 0 1"/>
-  </joint>
-  <link name="wheel_left_link">
-    <visual>
-      <origin xyz="0 0 0.015" rpy="0 0 0"/>
-      <geometry>
-        <mesh filename="package://${package_name}/meshes/wheel_ring.stl" scale="1 1 1"/>
-      </geometry>
-      <material name="white"/> <!-- Color in Rviz2 (inside visual tag) -->
-    </visual>
-    <collision>
-      <origin xyz="0 0 0" rpy="0 0 0"/>
-      <geometry>
-        <cylinder length="${wheelThickness}" radius="${wheelDiameter/2}"/>
-      </geometry>
-    </collision>
-    <inertial>
-      <origin xyz="0 0 0" />
-      <mass value="5" />
-      <inertia ixx="0.0135417" ixy="0.0" ixz="0.0"  iyy="0.0135417" iyz="0.0"  izz="0.025" />
-      </inertial>
-  </link>
-  <joint name="wheel_right_joint" type="continuous">
-    <parent link="base_link"/>
-    <child link="wheel_right_link"/>
-    <origin xyz="0 ${-wheelSeparation/2} ${wheelDiameter/2-base_elevation}" rpy="${-PI/2} 0 0"/>
-    <axis xyz="0 0 1"/>
-  </joint>
-  <link name="wheel_right_link">
-    <visual>
-      <origin xyz="0 0 -0.015" rpy="${PI} 0 0"/> <!-- -z and r=PI for the other wheel -->
-      <geometry>
-        <mesh filename="package://${package_name}/meshes/wheel_ring.stl" scale="1 1 1"/>
-      </geometry>
-      <material name="white"/> <!-- Color in Rviz2 (inside visual tag) -->
-    </visual>
-    <collision>
-      <origin xyz="0 0 0" rpy="0 0 0"/>
-      <geometry>
-        <cylinder length="${wheelThickness}" radius="${wheelDiameter/2}"/>
-      </geometry>
-    </collision>
-    <inertial>
-      <origin xyz="0 0 0" />
-      <mass value="5" />
-      <inertia ixx="0.0135417" ixy="0.0" ixz="0.0"  iyy="0.0135417" iyz="0.0"  izz="0.025" />
-    </inertial>
-  </link>
-  <!-- Caster wheel definition (joints and links) -->
-  <joint name="caster_base_joint" type="fixed">
-    <!--origin xyz="-0.104 0 0.015" rpy="0 0 ${PI}" /-->
-    <origin xyz="-0.135 -0.01 0.006" rpy="0 ${PI} ${PI}" />
-    <parent link="base_link" />
-    <!--child link="caster_base_link" /-->
-    <child link="caster_wheel_link" />
-    <!--axis xyz="0 0 1" /-->
-    <!--dynamics damping="0.001" fricction="0.001"/-->
-  </joint>
-  <link name="caster_wheel_link">
-    <visual>
-      <origin xyz="0 0 0" rpy="0 0 0" />
-      <geometry>
-        <mesh filename="package://${package_name}/meshes/bolaloca.stl" scale="0.001 0.001 0.001"/>
-      </geometry>
-    </visual>
-    <collision>
-      <origin xyz="0 0 0" rpy="0 0 0" />
-      <geometry>
-        <!--cylinder length="0.01" radius="0.015" /-->
-        <box size="0.01 0.1 0.03"/>
-      </geometry>
-    </collision>
-    <inertial>
-      <origin xyz="6.93889390390723E-18 -2.62037475051713E-11 -2.77710070911708E-09" rpy="0 0 0" />
-      <mass value="0.08" />
-      <inertia ixx="0.0004" ixy="0" ixz="0" iyy="0.0004" iyz="0" izz="0.00001" />
-    </inertial>
-  </link>
-  <!-- CAMERA -->
-  <!-- ESTE FUNCIONA -->
-  <!--joint name="camera_joint" type="fixed">
-    <origin xyz="0.04 0.025 0.05" rpy="0 0 0"/>
-    <parent link="base_link"/>
-    <child link="camera_frame"/>
-  </joint-->
-  <joint name="camera_joint" type="revolute">
-    <parent link="base_link"/>
-    <child link="camera_frame"/>
-    <origin xyz="0.04 0.025 0.05" rpy="0 0 0"/>
-    <axis xyz="0 1 0"/>
-    <!--limit effort="0.0" lower="0.0" upper="3.14" velocity="0.0"/-->
-    <limit effort="2.0" lower="0.0" upper="3.14" velocity="1.0"/>
-    <dynamics damping="0.05" friction="0.05"/>
-  </joint>
-  <link name="camera_frame"> <!-- Important: Every visual, collision and inertial tag has its own origin -->
-    <visual>
-      <!--origin xyz="-0.033 0.0 0.04" rpy="0 0 ${PI}"/-->
-      <origin xyz="0.0 0.0 0.0 " rpy="0 0 ${-PI/2}"/>
-      <geometry>
-        <!--mesh filename="package://${package_name}/meshes/base_plate.stl" scale="1 1 1"/-->
-        <mesh filename="package://${package_name}/meshes/camara.stl" scale="0.001 0.001 0.001"/>
-      </geometry>
-      <material name="Blue"> <!-- Color in Rviz2 (inside visual tag) -->
-        <color rgba="${0/255} ${0/255} ${255/255} 1.0"/>
-      </material>
-    </visual>
-    <!-- NECESARIO AÑADIRLO PARA QUE GAZEBO NO NOS IGNORE-->
-    <!-- Collision tag added to stabilize the robot -->
-    <collision>
-      <origin xyz="0.0 0.0 0.0 " rpy="0 0 ${-PI/2}"/>
-      <geometry>
-        <mesh filename="package://${package_name}/meshes/camara.stl" scale="0.001 0.001 0.001"/>
-      </geometry>
-    </collision>
-    <inertial>
-      <origin xyz="0.0 0.0 0.0" rpy="0 0 ${-PI/2}"/>
-      <mass value="0.03"/> <!--30g-->
-      <inertia ixx="0.01" ixy="0.0" ixz="0.0" iyy="0.005" iyz="0.0" izz="0.005"/>
-      </inertial>
-  </link>
-</robot>
+/home/juloau/Desktop/TFG/tfg-jlopez/code/ros2/src/pibotj/urdf/caster_diffbot.xacro

File: code/ros2/install/pibotj/share/pibotj/urdf/caster_diffbot_gz.xacro (robot description, xacro)
@@ -1,250 +1 @@
-<?xml version="1.0"?>
-<robot xmlns:xacro="http://ros.org/wiki/xacro">
-<!-- http://wiki.ros.org/simulator_gazebo/Tutorials/ListOfMaterials -->
-  <xacro:arg name="base_color"    default="Blue"/>
-  <!-- Custom color (for RViz) -->
-  <material name="white">
-    <color rgba="${250/255} ${250/255} ${250/255} 1.0"/>
-  </material>
-  <gazebo reference="base_link">
-    <material>Gazebo/$(arg base_color)</material> <!-- Color of the base link in Gazebo -->
-  </gazebo>
-  <gazebo reference="wheel_left_link">
-    <mu1>0.1</mu1>
-    <mu2>0.1</mu2>
-    <kp>500000.0</kp>
-    <kd>10.0</kd>
-    <minDepth>0.001</minDepth>
-    <maxVel>0.1</maxVel>
-    <fdir1>1 0 0</fdir1>
-    <material>Gazebo/DarkGrey</material>
-  </gazebo>
-  <gazebo reference="wheel_right_link">
-    <mu1>0.1</mu1>
-    <mu2>0.1</mu2>
-    <kp>500000.0</kp>
-    <kd>10.0</kd>
-    <minDepth>0.001</minDepth>
-    <maxVel>0.1</maxVel>
-    <fdir1>1 0 0</fdir1>
-    <material>Gazebo/DarkGrey</material>
-  </gazebo>
-  <!--gazebo reference="caster_base_link">
-    <mu1>0.1</mu1>
-    <mu2>0.1</mu2>
-    <kp>1000000</kp>
-    <kd>100.0</kd>
-    <minDepth>0.001</minDepth>
-    <maxVel>1.0</maxVel>
-    <material>Gazebo/$(arg base_color)</material>
-  </gazebo-->
-  <gazebo reference="caster_wheel_link">
-    <mu1>0.1</mu1>
-    <mu2>0.1</mu2>
-    <kp>1000000</kp>
-    <kd>100.0</kd>
-    <minDepth>0.001</minDepth>
-    <maxVel>1.0</maxVel>
-    <material>Gazebo/White</material>
-  </gazebo>
-  <!-- Plugins for a differential drive mobile robot in Gazebo with ROS 2 -->
-  <!-- 'libgazebo_ros_diff_drive.so' & 'libgazebo_ros_joint_state_publisher' -->
-  <gazebo>
-    <plugin name="diff_drive" filename="libgazebo_ros_diff_drive.so">
-      <!--num_wheel_pairs>2</num_wheel_pairs--> <!-- repeat 'left_joint' and 'right_joint' tags -->
-      <!-- robot does not respond as desired but all wheels rotate -->
-      <left_joint>wheel_left_joint</left_joint>
-      <right_joint>wheel_right_joint</right_joint>
-      <command_topic>cmd_vel</command_topic>
-      <!-- kinematics -->
-      <wheel_separation>${wheelSeparation}</wheel_separation>
-      <wheel_diameter>${wheelDiameter}</wheel_diameter>
-      <max_wheel_torque>20</max_wheel_torque>
-      <max_wheel_acceleration>10.0</max_wheel_acceleration>
-      <!-- odometry  -->
-      <odometry_topic>odom</odometry_topic>
-      <odometry_frame>odom</odometry_frame>
-      <robot_base_frame>base_footprint</robot_base_frame>
-      <odometry_source>1</odometry_source> <!-- 1=world or 0=encoder -->
-      <publish_odom>true</publish_odom>
-      <publish_odom_tf>true</publish_odom_tf>
-      <publish_wheel_tf>true</publish_wheel_tf>
-      <update_rate>30</update_rate>
-      <covariance_x>0.1</covariance_x>
-      <covariance_y>0.1</covariance_y>
-      <covariance_yaw>0.09</covariance_yaw>
-    </plugin>
-  </gazebo>
-  <gazebo>
-    <plugin name="diff_joint_state" filename="libgazebo_ros_joint_state_publisher.so">
-      <ros>
-        <!-- <namespace>/</namespace> -->
-        <remapping>~/out:=joint_states</remapping>
-      </ros>
-      <update_rate>30</update_rate>
-      <!-- list of mobile joints -->
-      <joint_name>wheel_left_joint</joint_name>
-      <joint_name>wheel_right_joint</joint_name>
-      <!-- camera HA SIDO NECESARIO INCLUIRLO AQUÍ SINO NO LO DETECTA RVIZ CORRECTAMENTE-->
-      <joint_name>camera_joint</joint_name>
-    </plugin>
-  </gazebo>
-  <!-- ******************** SENSORS PLUGINS ******************** -->
-  <!-- IMU -->
-  <!--gazebo reference="imu_link">
-    <sensor name="imu" type="imu">
-      <visualize>true</visualize>
-      <always_on>true</always_on>
-      <update_rate>30</update_rate>
-      <plugin name="imu_plugin" filename="libgazebo_ros_imu_sensor.so">
-        <ros-->
-          <!--namespace>/</namespace-->
-          <!--remapping>~/out:=imu</remapping>
-        </ros>
-        <initial_orientation_as_reference>false</initial_orientation_as_reference>
-      </plugin>
-      <imu>
-     	<angular_velocity>
-     	  <x>
-     	    <noise type="gaussian">
-              <mean>0.0</mean>
-              <stddev>2e-4</stddev>
-              <bias_mean>0.0000075</bias_mean>
-              <bias_stddev>0.0000008</bias_stddev>
-            </noise>
-          </x>
-          <y>
-            <noise type="gaussian">
-              <mean>0.0</mean>
-              <stddev>2e-4</stddev>
-              <bias_mean>0.0000075</bias_mean>
-              <bias_stddev>0.0000008</bias_stddev>
-            </noise>
-          </y>
-          <z>
-            <noise type="gaussian">
-              <mean>0.0</mean>
-              <stddev>2e-4</stddev>
-              <bias_mean>0.0000075</bias_mean>
-              <bias_stddev>0.0000008</bias_stddev>
-            </noise>
-          </z>
-        </angular_velocity>
-        <linear_acceleration>
-          <x>
-            <noise type="gaussian">
-              <mean>0.0</mean>
-              <stddev>1.7e-2</stddev>
-              <bias_mean>0.1</bias_mean>
-              <bias_stddev>0.001</bias_stddev>
-            </noise>
-          </x>
-          <y>
-            <noise type="gaussian">
-              <mean>0.0</mean>
-              <stddev>1.7e-2</stddev>
-              <bias_mean>0.1</bias_mean>
-              <bias_stddev>0.001</bias_stddev>
-            </noise>
-          </y>
-          <z>
-            <noise type="gaussian">
-              <mean>0.0</mean>
-              <stddev>1.7e-2</stddev>
-              <bias_mean>0.1</bias_mean>
-              <bias_stddev>0.001</bias_stddev>
-            </noise>
-          </z>
-        </linear_acceleration>
-      </imu>
-    </sensor>
-  </gazebo-->
-  <!-- LIDAR -->
-  <!--gazebo reference="lidar_link">
-    <material>Gazebo/Black</material>
-    <sensor type="ray" name="lidar">
-      <pose>0 0 0 0 0 0</pose>
-      <visualize>false</visualize>
-      <always_on>true</always_on>
-      <update_rate>10</update_rate>
-      <ray>
-        <scan>
-          <horizontal>
-            <samples>360</samples>
-            <resolution>1</resolution>
-            <min_angle>${-PI}</min_angle>
-            <max_angle>${PI}</max_angle>
-          </horizontal>
-        </scan>
-        <range>
-          <min>0.1</min>
-          <max>2.5</max>
-          <resolution>0.017453</resolution>
-        </range>
-        <noise>
-          <type>gaussian</type>
-          <mean>0.0</mean>
-          <stddev>0.01</stddev>
-        </noise>
-      </ray>
-      <plugin name="laser_plugin" filename="libgazebo_ros_ray_sensor.so">
-        <ros-->
-            <!--namespace>/</namespace-->
-            <!--remapping>~/out:=scan</remapping>
-        </ros-->
-        <!--topic_name>scan</topic_name-->
-        <!--output_type>sensor_msgs/LaserScan</output_type>
-        <frame_name>lidar_link</frame_name>
-      </plugin>
-    </sensor>
-  </gazebo-->
-  <!-- MONOCULAR CAMERA -->
-<gazebo reference="camera_joint">
-  <plugin name="camera_joint_control" filename="libgazebo_ros_joint_control.so">
-    <ros>
-      <namespace>/</namespace>
-      <remapping>~/command:=/camera_joint/command</remapping>
-    </ros>
-    <joint_name>camera_joint</joint_name>
-    <update_rate>30</update_rate>
-  </plugin>
-</gazebo>
-  <gazebo reference="camera_frame">
-    <material>Gazebo/Blue</material>
-    <sensor type="camera" name="camera">
-      <always_on>true</always_on>
-      <update_rate>30.0</update_rate>
-      <visualize>false</visualize>
-      <camera>
-        <horizontal_fov>1.085595</horizontal_fov>
-        <image>
-          <width>640</width>
-          <height>480</height>
-          <format>R8G8B8</format>
-        </image>
-        <clip>
-          <near>0.05</near>
-          <far>8.0</far>
-        </clip>
-        <distortion>
-         <k1>0.0</k1>
-         <k2>0.0</k2>
-         <k3>0.0</k3>
-         <p1>0.0</p1>
-         <p2>0.0</p2>
-         <center>0.5 0.5</center>
-       </distortion>
-      </camera>
-        <plugin name="camera_plugin" filename="libgazebo_ros_camera.so">
-            <ros>
-                <namespace>/</namespace>
-                <remapping>~/image_raw:=image_raw</remapping>
-                <remapping>~/camera_info:=camera_info</remapping>
-            </ros>
-            <camera_name>camera</camera_name>
-            <frame_name>camera_frame</frame_name>
-            <hack_baseline>0.2</hack_baseline>
-        </plugin>
-    </sensor>
-  </gazebo>
-</robot>
+/home/juloau/Desktop/TFG/tfg-jlopez/code/ros2/src/pibotj/urdf/caster_diffbot_gz.xacro

File: code/ros2/install/pibotj/share/pibotj/urdf/the_simplest_diffbot.xacro (robot description, xacro)
@@ -1,107 +1 @@
-<?xml version="1.0"?>
-<robot name="the_simplest_diffbot" xmlns:xacro="http://ros.org/wiki/xacro">
-  <xacro:include filename="$(find pibotj)/urdf/the_simplest_diffbot_gz.xacro"/>
-  <link name="base_footprint"/>
-  <joint name="base_joint" type="fixed">
-    <parent link="base_footprint"/>
-    <child link="base_link"/>
-    <origin xyz="0 0 0.01" rpy="0 0 0"/>
-  </joint>
-  <link name="base_link"> <!-- Important: Every visual, collision and inertial tag has its own origin -->
-    <visual>
-      <origin xyz="-0.033 0.0 0.04" rpy="0 0 0"/>
-      <geometry>
-        <box size="0.2 0.1 0.06"/>
-      </geometry>
-    </visual>
-    <collision>
-      <origin xyz="-0.033 0 0.04" rpy="0 0 0"/>
-      <geometry>
-        <box size="0.2 0.1 0.06"/>
-      </geometry>
-    </collision>
-    <inertial>
-      <origin xyz="0 0 0.06" rpy="0 0 0"/>
-      <mass value="10"/>
-      <inertia ixx="0.333333" ixy="0.0" ixz="0.0"  iyy="0.333333" iyz="0.0"  izz="0.6" />
-    </inertial>
-  </link>
-  <!-- Wheels definition (joints and links) -->
-  <joint name="wheel_left_joint" type="continuous">
-    <parent link="base_link"/>
-    <child link="wheel_left_link"/>
-    <origin xyz="0 0.065 0.025" rpy="-1.57 0 0"/> <!-- in rad -->
-    <axis xyz="0 0 1"/>
-  </joint>
-  <link name="wheel_left_link">
-    <visual>
-      <origin xyz="0 0 0.015" rpy="0 0 0"/>
-      <geometry>
-        <cylinder length="0.024" radius="0.035"/>
-      </geometry>
-    </visual>
-    <collision>
-      <origin xyz="0 0 0" rpy="0 0 0"/>
-      <geometry>
-        <cylinder length="0.024" radius="0.035"/>
-      </geometry>
-    </collision>
-    <inertial>
-      <origin xyz="0 0 0" />
-      <mass value="5" />
-      <inertia ixx="0.0135417" ixy="0.0" ixz="0.0"  iyy="0.0135417" iyz="0.0"  izz="0.025" />
-      </inertial>
-  </link>
-  <joint name="wheel_right_joint" type="continuous">
-    <parent link="base_link"/>
-    <child link="wheel_right_link"/>
-    <origin xyz="0 -0.065 0.025" rpy="-1.57 0 0"/>
-    <axis xyz="0 0 1"/>
-  </joint>
-  <link name="wheel_right_link">
-    <visual>
-      <origin xyz="0 0 -0.015" rpy="0 0 0"/>
-      <geometry>
-        <cylinder length="0.024" radius="0.035"/>
-      </geometry>
-    </visual>
-    <collision>
-      <origin xyz="0 0 0" rpy="0 0 0"/>
-      <geometry>
-        <cylinder length="0.024" radius="0.035"/>
-      </geometry>
-    </collision>
-    <inertial>
-      <origin xyz="0 0 0" />
-      <mass value="5" />
-      <inertia ixx="0.0135417" ixy="0.0" ixz="0.0"  iyy="0.0135417" iyz="0.0"  izz="0.025" />
-    </inertial>
-  </link>
-  <!-- Caster wheel definition (joint and link) -->
-  <joint name="caster_base_joint" type="fixed">
-    <origin xyz="-0.1 0 0.001" rpy="0 0 0" /> <!-- a small vertical offset is required -->
-    <parent link="base_link" />
-    <child link="caster_base_link" />
-  </joint>
-  <link name="caster_base_link">
-    <visual>
-      <origin xyz="0 0 0" rpy="0 0 0" />
-      <geometry>
-        <sphere radius="0.01"/>
-      </geometry>
-    </visual>
-    <collision>
-      <origin xyz="0 0 0" rpy="0 0 0"/>
-      <geometry>
-        <sphere radius="0.01"/>
-      </geometry>
-    </collision>
-    <collision>
-      <origin xyz="0.17 0 0" rpy="0 0 0"/>
-      <geometry>
-        <sphere radius="0.01"/>
-      </geometry>
-    </collision>
-    <!-- Inertial tag is optional for this case -->
-  </link>
-</robot>
+/home/juloau/Desktop/TFG/tfg-jlopez/code/ros2/src/pibotj/urdf/the_simplest_diffbot.xacro

File: code/ros2/install/pibotj/share/pibotj/urdf/the_simplest_diffbot_gz.xacro (robot description, xacro)
@@ -1,71 +1 @@
-<?xml version="1.0"?>
-<robot xmlns:xacro="http://ros.org/wiki/xacro">
-<!-- http://wiki.ros.org/simulator_gazebo/Tutorials/ListOfMaterials -->
-  <gazebo reference="base_link">
-    <material>Gazebo/Blue</material> <!-- Color of the base link in Gazebo -->
-  </gazebo>
-  <gazebo reference="wheel_left_link">
-    <mu1>0.1</mu1>
-    <mu2>0.1</mu2>
-    <kp>500000.0</kp>
-    <kd>10.0</kd>
-    <minDepth>0.001</minDepth>
-    <maxVel>0.1</maxVel>
-    <fdir1>1 0 0</fdir1>
-    <material>Gazebo/DarkGrey</material>
-  </gazebo>
-  <gazebo reference="wheel_right_link">
-    <mu1>0.1</mu1>
-    <mu2>0.1</mu2>
-    <kp>500000.0</kp>
-    <kd>10.0</kd>
-    <minDepth>0.001</minDepth>
-    <maxVel>0.1</maxVel>
-    <fdir1>1 0 0</fdir1>
-    <material>Gazebo/DarkGrey</material>
-  </gazebo>
-  <gazebo reference="caster_base_link">
-    <mu1>0.1</mu1>
-    <mu2>0.1</mu2>
-    <kp>1000000</kp>
-    <kd>100.0</kd>
-    <minDepth>0.001</minDepth>
-    <maxVel>1.0</maxVel>
-    <material>Gazebo/Red</material>
-  </gazebo>
-  <!-- Plugins for a differential drive mobile robot in Gazebo with ROS 2 -->
-  <!-- 'libgazebo_ros_diff_drive.so' & 'libgazebo_ros_joint_state_publisher' -->
-  <gazebo>
-    <plugin name="diff_drive" filename="libgazebo_ros_diff_drive.so">
-      <left_joint>wheel_left_joint</left_joint>
-      <right_joint>wheel_right_joint</right_joint>
-      <command_topic>cmd_vel</command_topic>
-      <!-- kinematics -->
-      <wheel_separation>0.13</wheel_separation>
-      <wheel_diameter>0.07</wheel_diameter>
-      <max_wheel_torque>20</max_wheel_torque>
-      <max_wheel_acceleration>10.0</max_wheel_acceleration>
-      <!-- odometry  -->
-      <odometry_topic>odom</odometry_topic>
-      <odometry_frame>odom</odometry_frame>
-      <robot_base_frame>base_footprint</robot_base_frame>
-      <odometry_source>1</odometry_source>
-      <publish_odom>true</publish_odom>
-      <publish_odom_tf>true</publish_odom_tf>
-      <publish_wheel_tf>false</publish_wheel_tf>
-      <update_rate>30</update_rate>
-    </plugin>
-  </gazebo>
-  <gazebo>
-    <plugin name="diff_joint_state" filename="libgazebo_ros_joint_state_publisher.so">
-      <ros>
-        <!-- <namespace>/</namespace> -->
-        <remapping>~/out:=joint_states</remapping>
-      </ros>
-      <update_rate>30</update_rate>
-      <!-- list of mobile joints -->
-      <joint_name>wheel_left_joint</joint_name>
-      <joint_name>wheel_right_joint</joint_name>
-    </plugin>
-  </gazebo>
-</robot>
+/home/juloau/Desktop/TFG/tfg-jlopez/code/ros2/src/pibotj/urdf/the_simplest_diffbot_gz.xacro
