Commit message: init gazebo

File: code/ros2/src/pibotj/urdf/caster_diffbot.xacro (robot description, xacro)
@@ -1,5 +1,5 @@
 <?xml version="1.0"?>
 <robot name="caster_diffbot" xmlns:xacro="http://ros.org/wiki/xacro">
-  <xacro:property name="package_name" value="pibotj_description"/>
+  <xacro:property name="package_name" value="pibotj"/>
   <xacro:property name="PI" value="3.14159265"/>
   <xacro:property name="wheelSeparation" value="0.13"/>

File: code/ros2/src/pibotj/urdf/the_simplest_diffbot.xacro (robot description, xacro)
@@ -1,5 +1,5 @@
 <?xml version="1.0"?>
 <robot name="the_simplest_diffbot" xmlns:xacro="http://ros.org/wiki/xacro">
-  <xacro:include filename="$(find pibotj_description)/urdf/the_simplest_diffbot_gz.xacro"/>
+  <xacro:include filename="$(find pibotj)/urdf/the_simplest_diffbot_gz.xacro"/>
   <link name="base_footprint"/>
   <joint name="base_joint" type="fixed">

Commit message: added images and updated pibotj

File: code/ros2/src/pibotj/urdf/caster_diffbot.xacro (robot description, xacro)
@@ -112,23 +112,4 @@
     <!--dynamics damping="0.001" fricction="0.001"/-->
   </joint>
-  <!--link name="caster_base_link">
-    <visual>
-      <origin xyz="0 0 0.015" rpy="${-PI} 0 0" />
-      <geometry>
-        <mesh filename="package://${package_name}/meshes/base_caster.stl" />
-      </geometry>
-    </visual>
-    <inertial>
-      <origin xyz="0 0 0" rpy="0 0 0" />
-      <mass value="0.5" />
-      <inertia ixx="0.00004" ixy="0" ixz="0" iyy="0.00004" iyz="0" izz="0.00001" />
-    </inertial>
-  </link-->
-  <!--joint name="caster_wheel_joint" type="fixed">
-    <origin xyz="0.015014 -0.00012272 -0.01" rpy="0 ${-PI/2} ${PI/2}" />
-    <parent link="caster_base_link" />
-    <child link="caster_wheel_link" /-->
-    <!--axis xyz="0 0 1" /-->
-  <!--/joint-->
   <link name="caster_wheel_link">
     <visual>
@@ -151,26 +132,4 @@
     </inertial>
   </link>
-  <!-- ******************** SENSORS DEFINITION ******************** -->
-  <!-- IMU -->
-  <!--joint name="imu_joint" type="fixed">
-    <parent link="base_link"/>
-    <child link="imu_link"/>
-    <origin xyz="0 0 0" rpy="0 0 0"/>
-  </joint>
-  <link name="imu_link" /-->
-  <!-- LIDAR -->
-  <!--joint name="lidar_joint" type="fixed">
-    <parent link="base_link"/>
-    <child link="lidar_link"/>
-    <origin xyz="-0.04 0 0.07" rpy="0 0 0"/>
-  </joint>
-  <link name="lidar_link">
-    <visual>
-      <origin xyz="0 0 0" rpy="0 0 0"/>
-      <geometry>
-        <cylinder length="0.05" radius="0.03" />
-      </geometry>
-    </visual>
-  </link-->
   <!-- CAMERA -->
   <!-- ESTE FUNCIONA -->
@@ -185,5 +144,6 @@
     <origin xyz="0.04 0.025 0.05" rpy="0 0 0"/>
     <axis xyz="0 1 0"/>
-    <limit effort="0.0" lower="0.0" upper="0.0" velocity="0.0"/>
+    <!--limit effort="0.0" lower="0.0" upper="3.14" velocity="0.0"/-->
+    <limit effort="2.0" lower="0.0" upper="3.14" velocity="1.0"/>
     <dynamics damping="0.05" friction="0.05"/>
   </joint>
@@ -214,22 +174,3 @@
       </inertial>
   </link>
-  <!--joint name="logo_joint" type="fixed">
-    <parent link="base_footprint"/>
-    <child link="logo_link"/>
-    <origin xyz="-0.09 0.0 0.05" rpy="0 0 0"/>
-  </joint-->
-  <!--link name="logo_link">
-    <visual>
-      <origin xyz="0 0 0" rpy="0 0 ${PI}"/>
-      <geometry>
-        <mesh filename="package://${package_name}/roboticaposgrado/meshes/RP_logo.dae" scale="0.2 0.2 0.2"/>
-      </geometry>
-    </visual>
-    <collision>
-      <origin xyz="0 0 0.05" rpy="0 0 0"/>
-      <geometry>
-        <box size="0.01 0.1 0.1"/>
-      </geometry>
-    </collision>
-  </link-->
 </robot>

File: code/ros2/src/pibotj/urdf/caster_diffbot_gz.xacro (robot description, xacro)
@@ -200,14 +200,14 @@
   </gazebo-->
   <!-- MONOCULAR CAMERA -->
-<!--gazebo reference="camera_joint">
+<gazebo reference="camera_joint">
   <plugin name="camera_joint_control" filename="libgazebo_ros_joint_control.so">
     <ros>
       <namespace>/</namespace>
-      <remapping>~/command:=camera_joint/command</remapping>
+      <remapping>~/command:=/camera_joint/command</remapping>
     </ros>
     <joint_name>camera_joint</joint_name>
     <update_rate>30</update_rate>
   </plugin>
-</gazebo-->
+</gazebo>
   <gazebo reference="camera_frame">
     <material>Gazebo/Blue</material>

Commit message: working pibotj with camera rotation

File: code/ros2/src/pibotj/urdf/caster_diffbot.xacro (robot description, xacro)
@@ -143,5 +143,5 @@
     <child link="camera_frame"/>
     <origin xyz="0.04 0.025 0.05" rpy="0 0 0"/>
-    <axis xyz="0 1 0"/>
+    <axis xyz="0 0 1"/>
     <!--limit effort="0.0" lower="0.0" upper="3.14" velocity="0.0"/-->
     <limit effort="2.0" lower="0.0" upper="3.14" velocity="1.0"/>
