Commit message: updated files

File: code/ros2/src/pibotj_r2c/description/ros2_control.xacro (robot description, xacro)
@@ -59,11 +59,4 @@
                 <state_interface name="position"/>
             </joint>
-            <!--joint name="camera_joint">
-                <command_interface name="velocity">
-                    <param name="min">-3</param>
-                    <param name="max">3</param>
-                </command_interface>
-                <state_interface name="velocity"/>
-            </joint-->
         </ros2_control>
     </xacro:if>
