Commit message: updated ros2 simulation robot

File: code/ros2/src/pibotj_r2c/description/gps.xacro (robot description, xacro)
@@ -9,10 +9,10 @@
         <visual>
              <geometry>
-                <mesh filename="package://pibotj_r2c/meshes/GY-NEO6MV2 NEO-6M.stl" scale="0.001 0.001 0.001"/>
+                <mesh filename="package://pibotj_r2c/meshes/GY-NEO6MV2NEO-6M.stl" scale="0.001 0.001 0.001"/>
             </geometry>
         </visual>
         <collision>
             <geometry>
-                <mesh filename="package://pibotj_r2c/meshes/GY-NEO6MV2 NEO-6M.stl" scale="0.001 0.001 0.001"/>
+                <mesh filename="package://pibotj_r2c/meshes/GY-NEO6MV2NEO-6M.stl" scale="0.001 0.001 0.001"/>
             </geometry>
         </collision>
