Commit message: added gazebo pibotj camera rotated

File: code/ros2/src/pibotj_r2c/description/camera.xacro (robot description, xacro)
@@ -59,11 +59,24 @@
         </inertial>
     </link>
+    <gazebo reference="camera_link">
+        <material>Gazebo/Blue</material>
+    </gazebo>
     <joint name="camera_optical_joint" type="fixed">
         <parent link="camera_link"/>
         <child link="camera_link_optical"/>
-        <origin xyz="0 0 0" rpy="${-pi/2} 0 ${-pi/2}"/>
+        <!--origin xyz="0.016 -0.018 0.02" rpy="0.8726 0 0"/-->
+         <origin xyz="0.016 -0.016 0.02" rpy="0 0.8726 0"/>
     </joint>
-    <link name="camera_link_optical"></link>
-    <gazebo reference="camera_link">
+    <!-- Cubo añadido donde va a ir la cámara-->
+    <link name="camera_link_optical">
+        <visual>
+            <!--origin xyz="0.016 -0.018 0.02" rpy="0.8726 0 0"/-->
+            <origin xyz="0 0 0" rpy="0 0 0"/>
+            <geometry>
+                <box size="0.01 0.01 0.01"/>
+            </geometry>
+        </visual>
+    </link>
+    <gazebo reference="camera_link_optical">
         <material>Gazebo/Blue</material>
         <sensor name="camera" type="camera">

File: code/ros2/src/pibotj_r2c/description/robot_core.xacro (robot description, xacro)
@@ -19,5 +19,5 @@
     <xacro:property name="wheelDiameter" value="0.07"/>
     <xacro:property name="wheelThickness" value="0.024"/>
-    <xacro:property name="base_elevation" value="0.01"/>
+    <xacro:property name="base_elevation" value="0.005"/>
     <material name="white">
         <color rgba="1 1 1 1" />
@@ -97,5 +97,6 @@
             <origin xyz="0 0 ${wheelDiameter-base_elevation}" rpy="0 0 0"/>
             <mass value="100"/>
-            <inertia ixx="0.333333" ixy="0.0" ixz="0.0"  iyy="0.333333" iyz="0.0"  izz="0.6" />
+            <!--inertia ixx="0.333333" ixy="0.0" ixz="0.0"  iyy="0.333333" iyz="0.0"  izz="0.6" /-->
+            <inertia ixx="3.375" ixy="0.0" ixz="0.0" iyy="0.808" iyz="0.0" izz="2.833" />
          </inertial>
     </link>
@@ -129,5 +130,5 @@
             <origin xyz="0 0 0.015" rpy="0 0 0"/>
             <geometry>
-                <mesh filename="package://pibotj_r2c/meshes/wheel_ring.stl" scale="1 1 1"/>
+                <mesh filename="package://pibotj_r2c/meshes/wheel_ring.stl" scale="0.9 0.9 0.9"/>
             </geometry>
             <material name="white"/> <!-- Color in Rviz2 (inside visual tag) -->
@@ -175,5 +176,5 @@
             <origin xyz="0 0 -0.015" rpy="${pi} 0 0"/> <!-- -z and r=PI for the other wheel -->
             <geometry>
-                <mesh filename="package://pibotj_r2c/meshes/wheel_ring.stl" scale="1 1 1"/>
+                <mesh filename="package://pibotj_r2c/meshes/wheel_ring.stl" scale="0.9 0.9 0.9"/>
             </geometry>
             <material name="white"/> <!-- Color in Rviz2 (inside visual tag) -->
@@ -231,6 +232,8 @@
         <inertial>
             <origin xyz="6.93889390390723E-18 -2.62037475051713E-11 -2.77710070911708E-09" rpy="0 0 0" />
-            <mass value="0.08" />
-            <inertia ixx="0.0004" ixy="0" ixz="0" iyy="0.0004" iyz="0" izz="0.00001" />
+            <!--mass value="0.08" /-->
+            <!--inertia ixx="0.0004" ixy="0" ixz="0" iyy="0.0004" iyz="0" izz="0.00001" /-->
+            <mass value="0.15" /> <!-- Aumentando la masa -->
+            <inertia ixx="0.0006" ixy="0" ixz="0" iyy="0.0006" iyz="0" izz="0.00002" /> <!-- Ajustando inercia acorde -->
         </inertial>
     </link>

Commit message: fixed rotation camera

File: code/ros2/src/pibotj_r2c/description/camera.xacro (robot description, xacro)
@@ -9,32 +9,18 @@
         <parent link="chassis"/>
         <child link="camera_link"/>
-       <!--origin xyz="0.276 0 0.181" rpy="0 0.18 0"/-->
-        <origin xyz="0.04 0.025 0.05" rpy="0 0 0"/>
+        <!--origin xyz="0.04 0.025 0.05" rpy="0 0 0"/-->
+        <!--origin xyz="0.03 0.01 0.05" rpy="0 0 0"/ last -->
+        <origin xyz="0.02 0.01 0.05" rpy="0 0 0"/>
         <axis xyz="0 0 1"/>
     <!--limit effort="0.0" lower="0.0" upper="3.14" velocity="0.0"/-->
-        <limit effort="2.0" lower="0.0" upper="3.14" velocity="1.0"/>
+        <limit effort="2.0" lower="${-pi/2}" upper="${pi/2}" velocity="0.5"/>
        <dynamics damping="0.05" friction="0.05"/>
     </joint>
     <link name="camera_link">
-        <!--visual>
-            <geometry>
-                <box size="0.010 0.03 0.03"/>
-            </geometry>
-            <material name="black"/>
-        </visual>
-        <collision>
-            <origin xyz="0.0 0.0 0.0 " rpy="0 0 ${-pi/2}"/>
-            <geometry>
-                <box size="0.010 0.03 0.03"/>
-            </geometry>
-        </collision>
-        <inertial>
-            <origin xyz="0.0 0.0 0.0" rpy="0 0 ${-pi/2}"/>
-            <mass value="0.03"/--> <!--30g-->
-            <!--inertia ixx="0.01" ixy="0.0" ixz="0.0" iyy="0.005" iyz="0.0" izz="0.005"/>
-            </inertial-->
         <visual>
             <!--origin xyz="-0.033 0.0 0.04" rpy="0 0 ${PI}"/-->
-            <origin xyz="0.0 0.0 0.0 " rpy="0 0 ${-pi/2}"/>
+            <!--origin xyz="0.0 0.0 0.0 " rpy="0 0 ${-pi/2}" last /-->
+            <!--origin xyz="0.01 0.01 0.0 " rpy="0 0 ${-pi/2}"/-->
+            <origin xyz="0.02 0.01 0.0 " rpy="0 0 ${-pi/2}"/>
             <geometry>
             <!--mesh filename="package://${package_name}/meshes/base_plate.stl" scale="1 1 1"/-->
@@ -66,5 +52,6 @@
         <child link="camera_link_optical"/>
         <!--origin xyz="0.016 -0.018 0.02" rpy="0.8726 0 0"/-->
-         <origin xyz="0.016 -0.016 0.02" rpy="0 0.8726 0"/>
+         <!--origin xyz="0.016 -0.016 0.02" rpy="0 0.8726 0"/-->
+        <origin xyz="0.04 -0.006 0.018" rpy="0 0.8726 0"/>
     </joint>
     <!-- Cubo añadido donde va a ir la cámara-->

File: code/ros2/src/pibotj_r2c/description/ros2_control.xacro (robot description, xacro)
@@ -54,9 +54,16 @@
             <joint name="camera_joint">
                 <command_interface name="position">
-                    <param name="min">-10</param>
-                    <param name="max">10</param>
+                    <param name="min">-3</param>
+                    <param name="max">3</param>
                 </command_interface>
                 <state_interface name="position"/>
             </joint>
+            <!--joint name="camera_joint">
+                <command_interface name="velocity">
+                    <param name="min">-3</param>
+                    <param name="max">3</param>
+                </command_interface>
+                <state_interface name="velocity"/>
+            </joint-->
         </ros2_control>
     </xacro:if>

Commit message: updated files

File: code/ros2/src/pibotj_r2c/description/camera.xacro (robot description, xacro)
@@ -1,17 +1,9 @@
 <?xml version="1.0"?>
 <robot xmlns:xacro="http://www.ros.org/wiki/xacro" >
-    <!--joint name="camera_joint" type="fixed">
-        <parent link="chassis"/>
-        <child link="camera_link"/>
-        <origin xyz="0.276 0 0.181" rpy="0 0.18 0"/>
-    </joint-->
     <joint name="camera_joint" type="revolute">
         <parent link="chassis"/>
         <child link="camera_link"/>
-        <!--origin xyz="0.04 0.025 0.05" rpy="0 0 0"/-->
-        <!--origin xyz="0.03 0.01 0.05" rpy="0 0 0"/ last -->
         <origin xyz="0.02 0.01 0.05" rpy="0 0 0"/>
         <axis xyz="0 0 1"/>
-    <!--limit effort="0.0" lower="0.0" upper="3.14" velocity="0.0"/-->
         <limit effort="2.0" lower="${-pi/2}" upper="${pi/2}" velocity="0.5"/>
        <dynamics damping="0.05" friction="0.05"/>
@@ -19,18 +11,13 @@
     <link name="camera_link">
         <visual>
-            <!--origin xyz="-0.033 0.0 0.04" rpy="0 0 ${PI}"/-->
-            <!--origin xyz="0.0 0.0 0.0 " rpy="0 0 ${-pi/2}" last /-->
-            <!--origin xyz="0.01 0.01 0.0 " rpy="0 0 ${-pi/2}"/-->
             <origin xyz="0.02 0.01 0.0 " rpy="0 0 ${-pi/2}"/>
             <geometry>
-            <!--mesh filename="package://${package_name}/meshes/base_plate.stl" scale="1 1 1"/-->
                 <mesh filename="package://pibotj_r2c/meshes/camara.stl" scale="0.001 0.001 0.001"/>
             </geometry>
-            <material name="Blue"> <!-- Color in Rviz2 (inside visual tag) -->
+            <material name="Blue"> <!-- Color en Rviz2-->
                 <color rgba="${0/255} ${0/255} ${255/255} 1.0"/>
             </material>
         </visual>
         <!-- NECESARIO AÑADIRLO PARA QUE GAZEBO NO NOS IGNORE-->
-        <!-- Collision tag added to stabilize the robot -->
         <collision>
             <origin xyz="0.0 0.0 0.0 " rpy="0 0 ${-pi/2}"/>
@@ -51,6 +38,4 @@
         <parent link="camera_link"/>
         <child link="camera_link_optical"/>
-        <!--origin xyz="0.016 -0.018 0.02" rpy="0.8726 0 0"/-->
-         <!--origin xyz="0.016 -0.016 0.02" rpy="0 0.8726 0"/-->
         <origin xyz="0.04 -0.006 0.018" rpy="0 0.8726 0"/>
     </joint>
@@ -58,5 +43,4 @@
     <link name="camera_link_optical">
         <visual>
-            <!--origin xyz="0.016 -0.018 0.02" rpy="0.8726 0 0"/-->
             <origin xyz="0 0 0" rpy="0 0 0"/>
             <geometry>

File: code/ros2/src/pibotj_r2c/description/gps.xacro (robot description, xacro)
@@ -9,10 +9,10 @@
         <visual>
              <geometry>
-                <mesh filename="package://pibotj_r2c/meshes/GY-NEO6MV2NEO-6M.stl" scale="0.001 0.001 0.001"/>
+                <mesh filename="package://pibotj_r2c/meshes/gps.stl" scale="0.001 0.001 0.001"/>
             </geometry>
         </visual>
         <collision>
             <geometry>
-                <mesh filename="package://pibotj_r2c/meshes/GY-NEO6MV2NEO-6M.stl" scale="0.001 0.001 0.001"/>
+                <mesh filename="package://pibotj_r2c/meshes/gps.stl" scale="0.001 0.001 0.001"/>
             </geometry>
         </collision>
@@ -20,39 +20,10 @@
     <gazebo reference="gps_frame">
         <material>Gazebo/Gray</material>
-        <!--sensor name="laser" type="ray">
-            <pose> 0 0 0 0 0 0 </pose>
-            <visualize>false</visualize>
-            <update_rate>10</update_rate>
-            <ray>
-                <scan>
-                    <horizontal>
-                        <samples>360</samples>
-                        <min_angle>-3.14</min_angle>
-                        <max_angle>3.14</max_angle>
-                    </horizontal>
-                </scan>
-                <range>
-                    <min>0.3</min>
-                    <max>12</max>
-                </range>
-            </ray>
-            <plugin name="laser_controller" filename="libgazebo_ros_ray_sensor.so">
-                <ros>
-                    <argument>~/out:=scan</argument>
-                </ros>
-                <output_type>sensor_msgs/LaserScan</output_type>
-                <frame_name>gps_frame</frame_name>
-            </plugin>
-        </sensor-->
         <sensor name="gps" type="gps">
         <pose>0 0 0 0 0 0</pose>
         <visualize>false</visualize>
-        <!--update_rate>1</update_rate--> <!-- Actualización a 1 Hz -->
         <always_on>true</always_on>
-        <update_rate>30</update_rate>
+        <update_rate>30</update_rate> <!-- Actualización a 1 Hz -->
             <plugin name="gps_controller" filename="libgazebo_ros_gps_sensor.so">
-                <!--ros>
-                    <argument>~/out:=fix</argument>
-                </ros-->
                 <ros>
                     <!-- publish to /gps/data -->

File: code/ros2/src/pibotj_r2c/description/robot.urdf.xacro (robot description, xacro)
@@ -12,5 +12,3 @@
     <xacro:include filename="gps.xacro" />
     <xacro:include filename="camera.xacro" />
-    <!-- <xacro:include filename="depth_camera.xacro" /> -->
-    <!--xacro:include filename="face.xacro" /-->
 </robot>

File: code/ros2/src/pibotj_r2c/description/robot_core.xacro (robot description, xacro)
@@ -1,19 +1,4 @@
 <?xml version="1.0"?>
 <robot xmlns:xacro="http://www.ros.org/wiki/xacro" >
-    <!--xacro:include filename="inertial_macros.xacro"/-->
-    <!--xacro:property name="chassis_length" value="0.335"/>
-    <xacro:property name="chassis_width" value="0.265"/>
-    <xacro:property name="chassis_height" value="0.138"/>
-    <xacro:property name="chassis_mass" value="1.0"/>
-    <xacro:property name="wheel_radius" value="0.033"/>
-    <xacro:property name="wheel_thickness" value="0.026"/>
-    <xacro:property name="wheel_mass" value="0.05"/>
-    <xacro:property name="wheel_offset_x" value="0.226"/>
-    <xacro:property name="wheel_offset_y" value="0.1485"/>
-    <xacro:property name="wheel_offset_z" value="0.01"/>
-    <xacro:property name="caster_wheel_radius" value="0.01"/>
-    <xacro:property name="caster_wheel_mass" value="0.01"/>
-    <xacro:property name="caster_wheel_offset_x" value="0.075"/>
-    <xacro:property name="caster_wheel_offset_z" value="${wheel_offset_z - wheel_radius + caster_wheel_radius}"/-->
     <xacro:property name="wheelSeparation" value="0.13"/>
     <xacro:property name="wheelDiameter" value="0.07"/>
@@ -50,29 +35,10 @@
         <parent link="base_link"/>
         <child link="chassis"/>
-        <!--origin xyz="${-wheel_offset_x} 0 ${-wheel_offset_z}"/-->
         <origin xyz="0 0 ${base_elevation}" rpy="0 0 0"/>
     </joint>
     <link name="chassis">
-        <!--visual>
-            <origin xyz="${chassis_length/2} 0 ${chassis_height/2}"/>
-            <geometry>
-                <box size="${chassis_length} ${chassis_width} ${chassis_height}"/>
-            </geometry>
-            <material name="orange"/>
-        </visual>
-        <collision>
-            <origin xyz="${chassis_length/2} 0 ${chassis_height/2}"/>
-            <geometry>
-                <box size="${chassis_length} ${chassis_width} ${chassis_height}"/>
-            </geometry>
-        </collision>
-        <xacro:inertial_box mass="0.5" x="${chassis_length}" y="${chassis_width}" z="${chassis_height}">
-            <origin xyz="${chassis_length/2} 0 ${chassis_height/2}" rpy="0 0 0"/>
-        </xacro:inertial_box-->
         <visual>
-            <!--origin xyz="-0.033 0.0 0.04" rpy="0 0 ${PI}"/-->
             <origin xyz="-0.17 -0.055 0.04" rpy="${-pi/2} 0 0"/>
             <geometry>
-            <!--mesh filename="package://${package_name}/meshes/base_plate.stl" scale="1 1 1"/-->
                 <mesh filename="package://pibotj_r2c/meshes/base.stl" scale="0.001 0.001 0.001"/>
             </geometry>
@@ -97,5 +63,4 @@
             <origin xyz="0 0 ${wheelDiameter-base_elevation}" rpy="0 0 0"/>
             <mass value="100"/>
-            <!--inertia ixx="0.333333" ixy="0.0" ixz="0.0"  iyy="0.333333" iyz="0.0"  izz="0.6" /-->
             <inertia ixx="3.375" ixy="0.0" ixz="0.0" iyy="0.808" iyz="0.0" izz="2.833" />
          </inertial>
@@ -108,23 +73,8 @@
         <parent link="base_link"/>
         <child link="left_wheel"/>
-        <!--origin xyz="0 ${wheel_offset_y} 0" rpy="-${pi/2} 0 0" /-->
         <origin xyz="0 ${wheelSeparation/2} ${wheelDiameter/2-base_elevation}" rpy="${-pi/2} 0 0"/>
         <axis xyz="0 0 1"/>
     </joint>
     <link name="left_wheel">
-        <!--visual>
-            <geometry>
-                <cylinder radius="${wheel_radius}" length="${wheel_thickness}"/>
-            </geometry>
-            <material name="blue"/>
-        </visual>
-        <collision>
-            <geometry>
-                <sphere radius="${wheel_radius}"/>
-            </geometry>
-        </collision>
-        <xacro:inertial_cylinder mass="${wheel_mass}" length="${wheel_thickness}" radius="${wheel_radius}">
-            <origin xyz="0 0 0" rpy="0 0 0"/>
-        </xacro:inertial_cylinder-->
         <visual>
             <origin xyz="0 0 0.015" rpy="0 0 0"/>
@@ -153,24 +103,8 @@
         <parent link="base_link"/>
         <child link="right_wheel"/>
-        <!--origin xyz="0 ${-wheel_offset_y} 0" rpy="${pi/2} 0 0" /-->
         <origin xyz="0 ${-wheelSeparation/2} ${wheelDiameter/2-base_elevation}" rpy="${-pi/2} 0 0"/>
-        <!--axis xyz="0 0 -1"/-->
         <axis xyz="0 0 1"/>
     </joint>
     <link name="right_wheel">
-        <!--visual>
-            <geometry>
-                <cylinder radius="${wheel_radius}" length="${wheel_thickness}"/>
-            </geometry>
-            <material name="blue"/>
-        </visual>
-        <collision>
-            <geometry>
-                <sphere radius="${wheel_radius}"/>
-            </geometry>
-        </collision>
-        <xacro:inertial_cylinder mass="${wheel_mass}" length="${wheel_thickness}" radius="${wheel_radius}">
-            <origin xyz="0 0 0" rpy="0 0 0"/>
-        </xacro:inertial_cylinder-->
         <visual>
             <origin xyz="0 0 -0.015" rpy="${pi} 0 0"/> <!-- -z and r=PI for the other wheel -->
@@ -178,5 +112,5 @@
                 <mesh filename="package://pibotj_r2c/meshes/wheel_ring.stl" scale="0.9 0.9 0.9"/>
             </geometry>
-            <material name="white"/> <!-- Color in Rviz2 (inside visual tag) -->
+            <material name="white"/> <!-- Color en Rviz2-->
         </visual>
         <collision>
@@ -199,22 +133,7 @@
         <parent link="chassis"/>
         <child link="caster_wheel"/>
-        <!--origin xyz="${caster_wheel_offset_x} 0 ${caster_wheel_offset_z}"/-->
         <origin xyz="-0.135 -0.01 0.006" rpy="0 ${pi} ${pi}" />
     </joint>
     <link name="caster_wheel">
-        <!--visual>
-            <geometry>
-                <sphere radius="${caster_wheel_radius}"/>
-            </geometry>
-            <material name="white"/>
-        </visual>
-        <collision>
-            <geometry>
-                <sphere radius="${caster_wheel_radius}"/>
-            </geometry>
-        </collision>
-        <xacro:inertial_sphere mass="${caster_wheel_mass}" radius="${caster_wheel_radius}">
-            <origin xyz="0 0 0" rpy="0 0 0"/>
-        </xacro:inertial_sphere-->
         <visual>
             <origin xyz="0 0 0" rpy="0 0 0" />
@@ -226,5 +145,4 @@
             <origin xyz="0 0 0" rpy="0 0 0" />
             <geometry>
-                <!--cylinder length="0.01" radius="0.015" /-->
                 <box size="0.01 0.1 0.03"/>
             </geometry>
@@ -232,8 +150,6 @@
         <inertial>
             <origin xyz="6.93889390390723E-18 -2.62037475051713E-11 -2.77710070911708E-09" rpy="0 0 0" />
-            <!--mass value="0.08" /-->
-            <!--inertia ixx="0.0004" ixy="0" ixz="0" iyy="0.0004" iyz="0" izz="0.00001" /-->
-            <mass value="0.15" /> <!-- Aumentando la masa -->
-            <inertia ixx="0.0006" ixy="0" ixz="0" iyy="0.0006" iyz="0" izz="0.00002" /> <!-- Ajustando inercia acorde -->
+            <mass value="0.15" />
+            <inertia ixx="0.0006" ixy="0" ixz="0" iyy="0.0006" iyz="0" izz="0.00002" />
         </inertial>
     </link>
