Commit message: updated puibotj_r2c

File: code/ros2/src/pibotj_r2c/description/robot.urdf.xacro (robot description, xacro)
@@ -1,13 +1,14 @@
 <?xml version="1.0"?>
 <robot xmlns:xacro="http://www.ros.org/wiki/xacro"  name="robot">
-    <xacro:arg name="use_ros2_control" default="true"/>
-    <xacro:arg name="sim_mode" default="false"/>
+    <!--xacro:arg name="use_ros2_control" default="true"/-->
+    <!--xacro:arg name="sim_mode" default="false"/-->
+    <!--xacro:arg name="sim_mode" default="true"/-->
     <xacro:include filename="robot_core.xacro" />
-    <xacro:if value="$(arg use_ros2_control)">
-        <xacro:include filename="ros2_control.xacro" />
-    </xacro:if>
-    <xacro:unless value="$(arg use_ros2_control)">
-        <xacro:include filename="gazebo_control.xacro" />
-    </xacro:unless>
+    <!--xacro:if value="$(arg use_ros2_control)"-->
+    <xacro:include filename="ros2_control.xacro" />
+    <!---/xacro:if-->
+    <!--xacro:unless value="$(arg use_ros2_control)"-->
+    <xacro:include filename="gazebo_control.xacro" />
+    <!--/xacro:unless-->
     <xacro:include filename="gps.xacro" />
     <xacro:include filename="camera.xacro" />

File: code/ros2/src/pibotj_r2c/description/robot_core.xacro (robot description, xacro)
@@ -150,5 +150,5 @@
         <inertial>
             <origin xyz="6.93889390390723E-18 -2.62037475051713E-11 -2.77710070911708E-09" rpy="0 0 0" />
-            <mass value="0.15" />
+            <mass value="10.0" />
             <inertia ixx="0.0006" ixy="0" ixz="0" iyy="0.0006" iyz="0" izz="0.00002" />
         </inertial>

File: code/ros2/src/pibotj_r2c/description/ros2_control.xacro (robot description, xacro)
@@ -1,5 +1,5 @@
 <?xml version="1.0"?>
 <robot xmlns:xacro="http://www.ros.org/wiki/xacro">
-    <xacro:unless value="$(arg sim_mode)">
+    <!--xacro:unless value="$(arg sim_mode)">
         <ros2_control name="RealRobot" type="system">
             <hardware>
@@ -30,35 +30,35 @@
             </joint>
         </ros2_control>
-    </xacro:unless>
-    <xacro:if value="$(arg sim_mode)">
-        <ros2_control name="GazeboSystem" type="system">
-            <hardware>
-                <plugin>gazebo_ros2_control/GazeboSystem</plugin>
-            </hardware>
-            <joint name="left_wheel_joint">
-                <command_interface name="velocity">
-                    <param name="min">-10</param>
-                    <param name="max">10</param>
-                </command_interface>
-                <state_interface name="velocity"/>
-                <state_interface name="position"/>
-            </joint>
-            <joint name="right_wheel_joint">
-                <command_interface name="velocity">
-                    <param name="min">-10</param>
-                    <param name="max">10</param>
-                </command_interface>
-                <state_interface name="velocity"/>
-                <state_interface name="position"/>
-            </joint>
-            <joint name="camera_joint">
-                <command_interface name="position">
-                    <param name="min">-3</param>
-                    <param name="max">3</param>
-                </command_interface>
-                <state_interface name="position"/>
-            </joint>
-        </ros2_control>
-    </xacro:if>
+    </xacro:unless-->
+    <!--xacro:if value="$(arg sim_mode)"-->
+    <ros2_control name="GazeboSystem" type="system">
+        <hardware>
+            <plugin>gazebo_ros2_control/GazeboSystem</plugin>
+        </hardware>
+        <joint name="left_wheel_joint">
+            <command_interface name="velocity">
+                <param name="min">-10</param>
+                <param name="max">10</param>
+            </command_interface>
+            <state_interface name="velocity"/>
+            <state_interface name="position"/>
+        </joint>
+        <joint name="right_wheel_joint">
+            <command_interface name="velocity">
+                <param name="min">-10</param>
+                <param name="max">10</param>
+            </command_interface>
+            <state_interface name="velocity"/>
+            <state_interface name="position"/>
+        </joint>
+        <joint name="camera_joint">
+            <command_interface name="position">
+                <param name="min">-3</param>
+                <param name="max">3</param>
+            </command_interface>
+            <state_interface name="position"/>
+        </joint>
+    </ros2_control>
+    <!--/xacro:if-->
     <gazebo>
         <plugin name="gazebo_ros2_control" filename="libgazebo_ros2_control.so">

Commit message: updated puibotj_r2c working  commented

File: code/ros2/src/pibotj_r2c/description/robot.urdf.xacro (robot description, xacro)
@@ -1,15 +1,7 @@
 <?xml version="1.0"?>
 <robot xmlns:xacro="http://www.ros.org/wiki/xacro"  name="robot">
-    <!--xacro:arg name="use_ros2_control" default="true"/-->
-    <!--xacro:arg name="sim_mode" default="false"/-->
-    <!--xacro:arg name="sim_mode" default="true"/-->
-    <xacro:include filename="robot_core.xacro" />
-    <!--xacro:if value="$(arg use_ros2_control)"-->
-    <xacro:include filename="ros2_control.xacro" />
-    <!---/xacro:if-->
-    <!--xacro:unless value="$(arg use_ros2_control)"-->
-    <!--xacro:include filename="gazebo_control.xacro" /-->
-    <!--/xacro:unless-->
-    <xacro:include filename="gps.xacro" />
-    <xacro:include filename="camera.xacro" />
+    <xacro:include filename="robot_core.xacro"/>
+    <xacro:include filename="ros2_control.xacro"/>
+    <xacro:include filename="gps.xacro"/>
+    <xacro:include filename="camera.xacro"/>
 </robot>

File: code/ros2/src/pibotj_r2c/description/robot_core.xacro (robot description, xacro)
@@ -8,7 +8,7 @@
         <color rgba="1 1 1 1" />
     </material>
-    <material name="orange">
+    <!--material name="orange">
         <color rgba="1 0.3 0.1 1"/>
-    </material>
+    </material-->
     <material name="blue">
         <color rgba="0.2 0.2 1 1"/>
@@ -17,8 +17,9 @@
         <color rgba="0 0 0 1"/>
     </material>
-    <material name="red">
+    <!--material name="red">
         <color rgba="1 0 0 1"/>
-    </material>
+    </material-->
     <!-- BASE LINK -->
+    <!-- se encuentra en el centro a la altura de la unión de las ruedas -->
     <link name="base_link">
     </link>
@@ -43,5 +44,5 @@
                 <mesh filename="package://pibotj_r2c/meshes/base.stl" scale="0.001 0.001 0.001"/>
             </geometry>
-            <material name="Blue"> <!-- Color in Rviz2 (inside visual tag) -->
+            <material name="blue">
                 <color rgba="${0/255} ${0/255} ${255/255} 1.0"/>
             </material>
@@ -82,5 +83,5 @@
                 <mesh filename="package://pibotj_r2c/meshes/wheel_ring.stl" scale="0.9 0.9 0.9"/>
             </geometry>
-            <material name="white"/> <!-- Color in Rviz2 (inside visual tag) -->
+            <material name="white"/>
         </visual>
         <collision>
@@ -108,9 +109,9 @@
     <link name="right_wheel">
         <visual>
-            <origin xyz="0 0 -0.015" rpy="${pi} 0 0"/> <!-- -z and r=PI for the other wheel -->
+            <origin xyz="0 0 -0.015" rpy="${pi} 0 0"/> <!-- -zy r=PI para la otra rueda-->
             <geometry>
                 <mesh filename="package://pibotj_r2c/meshes/wheel_ring.stl" scale="0.9 0.9 0.9"/>
             </geometry>
-            <material name="white"/> <!-- Color en Rviz2-->
+            <material name="white"/>
         </visual>
         <collision>

File: code/ros2/src/pibotj_r2c/description/ros2_control.xacro (robot description, xacro)
@@ -1,40 +1,12 @@
 <?xml version="1.0"?>
 <robot xmlns:xacro="http://www.ros.org/wiki/xacro">
-    <!--xacro:unless value="$(arg sim_mode)">
-        <ros2_control name="RealRobot" type="system">
-            <hardware>
-                <plugin>diffdrive_arduino/DiffDriveArduino</plugin>
-                <param name="left_wheel_name">left_wheel_joint</param>
-                <param name="right_wheel_name">right_wheel_joint</param>
-                <param name="loop_rate">30</param>
-                <param name="device">/dev/ttyUSB0</param>
-                <param name="baud_rate">57600</param>
-                <param name="timeout">1000</param>
-                <param name="enc_counts_per_rev">3436</param>
-            </hardware>
-            <joint name="left_wheel_joint">
-                <command_interface name="velocity">
-                    <param name="min">-10</param>
-                    <param name="max">10</param>
-                </command_interface>
-                <state_interface name="velocity"/>
-                <state_interface name="position"/>
-            </joint>
-            <joint name="right_wheel_joint">
-                <command_interface name="velocity">
-                    <param name="min">-10</param>
-                    <param name="max">10</param>
-                </command_interface>
-                <state_interface name="velocity"/>
-                <state_interface name="position"/>
-            </joint>
-        </ros2_control>
-    </xacro:unless-->
-    <!--xacro:if value="$(arg sim_mode)"-->
     <ros2_control name="GazeboSystem" type="system">
         <hardware>
-            <plugin>gazebo_ros2_control/GazeboSystem</plugin>
+            <plugin>gazebo_ros2_control/GazeboSystem</plugin>  <!-- Este es el Hardware Interface para el Controller Manager-->
+            <!-- Se ha llamado GazeboSystem pero se puede llamar de cualquier forma-->
         </hardware>
+        <!-- Es el momento de definir las joints que tiene nuestro harware interface GazeboSystem-->
         <joint name="left_wheel_joint">
+            <!-- Las ruedas se moverán usando velocidad-->
             <command_interface name="velocity">
                 <param name="min">-10</param>
@@ -52,4 +24,5 @@
             <state_interface name="position"/>
         </joint>
+        <!-- El motor de la cámara se moverá usando posición-->
         <joint name="camera_joint">
             <command_interface name="position">
@@ -60,5 +33,9 @@
         </joint>
     </ros2_control>
-    <!--/xacro:if-->
+    <!-- Plugin Gazebo que le dice a gazebo que use ros2 control-->
+    <!-- gazebo_ros2_control hace muchas cosas por nosotros, hace cosas de gazebo pero
+         tiene su propio controller manager -->
+    <!-- este controller manager es capaz de coger el URDF a través del \robot_state_publisher pero
+    necesitamos un .yaml que se llamará my_controllers-->
     <gazebo>
         <plugin name="gazebo_ros2_control" filename="libgazebo_ros2_control.so">
