Commit message: wip capitulo 6

File: code/ros2/src/pibotj_r2c/description/robot_core.xacro (robot description, xacro)
@@ -8,7 +8,4 @@
         <color rgba="1 1 1 1" />
     </material>
-    <!--material name="orange">
-        <color rgba="1 0.3 0.1 1"/>
-    </material-->
     <material name="blue">
         <color rgba="0.2 0.2 1 1"/>
@@ -17,7 +14,4 @@
         <color rgba="0 0 0 1"/>
     </material>
-    <!--material name="red">
-        <color rgba="1 0 0 1"/>
-    </material-->
     <!-- BASE LINK -->
     <!-- se encuentra en el centro a la altura de la unión de las ruedas -->
